Commit message: add 2d laser and differential driver

File: urdf/barista_robot_urdf.urdf (robot description, URDF)
Before this commit: robot barista_robot, 10 links, 8 joints
Links:
- removed link wheels
- link front_caster: geometry collision cylinder length=0.0352 radius=0.01; visual cylinder length=0.0352 radius=0.01
- link laser: geometry collision mesh filename=file:///home/user/ros2_ws/src/barista_robot_description/mes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 scale=1 1 1; visual mesh filename=file:///home/user/ros2_ws/src/barista_robot_description/mes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 scale=1 1 1
- link rear_caster: geometry collision cylinder length=0.0352 radius=0.01; visual cylinder length=0.0352 radius=0.01
Joints:
- joint base_link_left_standoff_joint: origin xyz=0 -0.125 0.155 rpy=0 0 0 -> xyz=0 0.125 0.155 rpy=0 0 0
- joint base_link_left_wheel_joint: origin xyz=0 -0.15 0.0 rpy=0 0 0 -> xyz=0 0.15 0.0 rpy=0 0 0
- joint base_link_right_standoff_joint: origin xyz=0 0.125 0.155 rpy=0 0 0 -> xyz=0 -0.125 0.155 rpy=0 0 0
- joint base_link_right_wheel_joint: origin xyz=0 0.15 0.0 rpy=0 0 0 -> xyz=0 -0.15 0.0 rpy=0 0 0
