Commit message: enable launching 2 robots

File: xacro/barista_robot_model.gazebo.xacro (robot description, xacro)
@@ -2,27 +2,28 @@
 <robot xmlns:xacro="http://www.ros.org/wiki/xacro">
     <xacro:macro name="gazebo_elements">
+        <xacro:arg name="tray_color_gazebo" default ="Blue" />
         <!-- Gazebo Properties -->
-        <gazebo reference="base_link">
+        <gazebo reference="$(arg robot_name)_base_link">
             <material>Gazebo/Black</material>
         </gazebo>
-        <gazebo reference="cup_holder">
-            <material>Gazebo/Blue</material>
+        <gazebo reference="$(arg robot_name)_cup_holder">
+            <material>Gazebo/$(arg tray_color_gazebo)</material>
         </gazebo>
-        <gazebo reference="left_wheel">
+        <gazebo reference="$(arg robot_name)_left_wheel">
             <material>Gazebo/Red</material>
             <mu1>1</mu1>
             <mu2>1</mu2>
         </gazebo>
-        <gazebo reference="right_wheel">
+        <gazebo reference="$(arg robot_name)_right_wheel">
             <material>Gazebo/Red</material>
             <mu1>1</mu1>
             <mu2>1</mu2>
         </gazebo>
-        <gazebo reference="front_caster">
+        <gazebo reference="$(arg robot_name)_front_caster">
             <mu1>0</mu1>
             <mu2>0</mu2>
             <material>Gazebo/Gray</material>
         </gazebo>
-        <gazebo reference="rear_caster">
+        <gazebo reference="$(arg robot_name)_rear_caster">
             <mu1>0</mu1>
             <mu2>0</mu2>
@@ -30,10 +31,35 @@
         </gazebo>
         <!-- Gazebo Plugins -->
+        <gazebo>
+    <plugin name="box_bot_joint_state" filename="libgazebo_ros_joint_state_publisher.so">
+      <ros>
+          <namespace>/$(arg robot_name)</namespace>
+          <remapping>~/out:=$(arg robot_name)/joint_states</remapping>
+      </ros>
+      <update_rate>30</update_rate>
+      <joint_name>$(arg robot_name)_base_link_base_footprint_joint</joint_name>
+      <joint_name>$(arg robot_name)_base_link_left_wheel_joint</joint_name>
+      <joint_name>$(arg robot_name)_base_link_right_wheel_joint</joint_name>
+      <joint_name>$(arg robot_name)_base_link_left_front_standoff_joint</joint_name>
+      <joint_name>$(arg robot_name)_base_link_left_rear_standoff_joint</joint_name>
+      <joint_name>$(arg robot_name)_base_link_right_front_standoff_joint</joint_name>
+      <joint_name>$(arg robot_name)_base_link_right_rear_standoff_joint</joint_name>
+      <joint_name>$(arg robot_name)_base_link_cup_holder_joint</joint_name>
+      <joint_name>$(arg robot_name)_base_link_front_caster_joint</joint_name>
+      <joint_name>$(arg robot_name)_base_link_rear_caster_joint</joint_name>
+      <joint_name>$(arg robot_name)_base_link_laser_joint</joint_name>
+    </plugin>
+  </gazebo>
         <!-- Robot differential driver -->
         <gazebo>
             <plugin filename="libgazebo_ros_diff_drive.so" name="differential_drive_controller">
+                <ros>
+                    <namespace>$(arg robot_name)</namespace>
+                    <!-- <remapping>/odom:=$(arg robot_name)/odom</remapping> -->
+                    <!-- <remapping>/cmd_vel:=$(arg robot_name)/cmd_vel</remapping> -->
+                </ros>
                 <update_rate>20</update_rate>
-                <left_joint>base_link_left_wheel_joint</left_joint>
-                <right_joint>base_link_right_wheel_joint</right_joint>
+                <left_joint>$(arg robot_name)_base_link_left_wheel_joint</left_joint>
+                <right_joint>$(arg robot_name)_base_link_right_wheel_joint</right_joint>
                 <wheel_separation>0.3</wheel_separation>
                 <wheel_diameter>0.0352</wheel_diameter>
@@ -44,14 +70,14 @@
                 <publish_odom>true</publish_odom>
                 <publish_odom_tf>true</publish_odom_tf>
-                <odometry_frame>odom</odometry_frame>
-                <command_topic>cmd_vel</command_topic>
-                <robot_base_frame>base_link</robot_base_frame>
+                <odometry_frame>$(arg robot_name)_odom</odometry_frame>
+                <!-- <command_topic>$(arg robot_name)/cmd_vel</command_topic> -->
+                <robot_base_frame>$(arg robot_name)_base_footprint</robot_base_frame>
             </plugin>
         </gazebo>
         <!-- Laser scan -->
-        <gazebo reference="base_link_laser_joint">
+        <gazebo reference="$(arg robot_name)_base_link_laser_joint">
             <preserveFixedJoint>true</preserveFixedJoint>
         </gazebo>
-        <gazebo reference="laser">
+        <gazebo reference="$(arg robot_name)_laser">
             <sensor type="ray" name="head_hokuyo_sensor">
                 <pose>0 0 0 0 0 0</pose>
@@ -80,5 +106,6 @@
                 <plugin name="laser" filename="libgazebo_ros_ray_sensor.so">
                     <ros>
-                        <remapping>/laser/out:=/scan</remapping>
+                        <namespace>$(arg robot_name)</namespace>
+                        <remapping>/$(arg robot_name)/laser/out:=/$(arg robot_name)/scan</remapping>
                     </ros>
                     <output_type>sensor_msgs/LaserScan</output_type>

File: xacro/barista_robot_model.urdf.xacro (robot description, xacro)
@@ -1,4 +1,7 @@
 <?xml version="1.0"?>
 <robot xmlns:xacro="http://www.ros.org/wiki/xacro" name="barista_robot">
+    <!-- default robot name -->
+    <xacro:arg name="robot_name" default ="barista_robot" />
+    <!-- includes -->
     <xacro:include filename="$(find barista_robot_description)/xacro/materials.xacro"/>
     <xacro:include filename="$(find barista_robot_description)/xacro/wheel.xacro"/>
@@ -24,6 +27,14 @@
     <!-- laser -->
     <xacro:arg name="include_laser" default="true"/>
+    <!-- base footprint -->
+    <link name="$(arg robot_name)_base_footprint">
+    </link>
+    <joint name="$(arg robot_name)_base_link_base_footprint_joint" type="fixed">
+        <origin rpy="0 0 0" xyz="0 0 -0.0352"/>
+        <parent link="$(arg robot_name)_base_footprint"/>
+        <child link="$(arg robot_name)_base_link"/>
+    </joint>
     <!-- Base link -->
-    <link name="base_link">
+    <link name="$(arg robot_name)_base_link">
         <collision>
             <origin xyz="0 0 0.0775"/>
@@ -46,75 +57,75 @@
     </link>
     <!-- left wheel -->
-    <xacro:wheel wheel_name="left_wheel" wheel_length="${wheel_length}" wheel_radius="${wheel_radius}" />
-    <joint name="base_link_left_wheel_joint" type="continuous">
-        <axis xyz="0 1 0" rpy="0 0 0" />
+    <xacro:wheel wheel_name="$(arg robot_name)_left_wheel" wheel_length="${wheel_length}" wheel_radius="${wheel_radius}" />
+    <joint name="$(arg robot_name)_base_link_left_wheel_joint" type="continuous">
+        <axis xyz="0 1 0" />
         <origin xyz="0 0.15 0.0" rpy="0 0 0" />
-        <parent link="base_link" />
-        <child link="left_wheel" />
+        <parent link="$(arg robot_name)_base_link" />
+        <child link="$(arg robot_name)_left_wheel" />
     </joint>
     <!-- right wheel -->
-    <xacro:wheel wheel_name="right_wheel" wheel_length="${wheel_length}" wheel_radius="${wheel_radius}" />
-    <joint name="base_link_right_wheel_joint" type="continuous">
-        <axis xyz="0 1 0" rpy="0 0 0" />
+    <xacro:wheel wheel_name="$(arg robot_name)_right_wheel" wheel_length="${wheel_length}" wheel_radius="${wheel_radius}" />
+    <joint name="$(arg robot_name)_base_link_right_wheel_joint" type="continuous">
+        <axis xyz="0 1 0" />
         <origin xyz="0 -0.15 0.0" rpy="0 0 0" />
-        <parent link="base_link" />
-        <child link="right_wheel" />
+        <parent link="$(arg robot_name)_base_link" />
+        <child link="$(arg robot_name)_right_wheel" />
     </joint>
     <!-- left-front standoff -->
-    <xacro:standoff standoff_name="left_front_standoff" standoff_length="${standoff_length}" standoff_radius="${standoff_radius}" />
-    <joint name="base_link_left_front_standoff_joint" type="fixed">
+    <xacro:standoff standoff_name="$(arg robot_name)_left_front_standoff" standoff_length="${standoff_length}" standoff_radius="${standoff_radius}" />
+    <joint name="$(arg robot_name)_base_link_left_front_standoff_joint" type="fixed">
         <origin rpy="0 0 0" xyz="0.025 0.125 0.155" />
-        <parent link="base_link" />
-        <child link="left_front_standoff" />
+        <parent link="$(arg robot_name)_base_link" />
+        <child link="$(arg robot_name)_left_front_standoff" />
     </joint>
     <!-- left-rear standoff -->
-    <xacro:standoff standoff_name="left_rear_standoff" standoff_length="${standoff_length}" standoff_radius="${standoff_radius}"/>
-    <joint name="base_link_left_rear_standoff_joint" type="fixed">
+    <xacro:standoff standoff_name="$(arg robot_name)_left_rear_standoff" standoff_length="${standoff_length}" standoff_radius="${standoff_radius}"/>
+    <joint name="$(arg robot_name)_base_link_left_rear_standoff_joint" type="fixed">
         <origin rpy="0 0 0" xyz="-0.025 0.125 0.155" />
-        <parent link="base_link" />
-        <child link="left_rear_standoff" />
+        <parent link="$(arg robot_name)_base_link" />
+        <child link="$(arg robot_name)_left_rear_standoff" />
     </joint>
     <!-- right-front standoff -->
-    <xacro:standoff standoff_name="right_front_standoff" standoff_length="${standoff_length}" standoff_radius="${standoff_radius}" />
-    <joint name="base_link_right_front_standoff_joint" type="fixed">
+    <xacro:standoff standoff_name="$(arg robot_name)_right_front_standoff" standoff_length="${standoff_length}" standoff_radius="${standoff_radius}" />
+    <joint name="$(arg robot_name)_base_link_right_front_standoff_joint" type="fixed">
         <origin rpy="0 0 0" xyz="0.025 -0.125 0.155" />
-        <parent link="base_link" />
-        <child link="right_front_standoff" />
+        <parent link="$(arg robot_name)_base_link" />
+        <child link="$(arg robot_name)_right_front_standoff" />
     </joint>
     <!-- right-rear standoff -->
-    <xacro:standoff standoff_name="right_rear_standoff" standoff_length="${standoff_length}" standoff_radius="${standoff_radius}" />
-    <joint name="base_link_right_rear_standoff_joint" type="fixed">
+    <xacro:standoff standoff_name="$(arg robot_name)_right_rear_standoff" standoff_length="${standoff_length}" standoff_radius="${standoff_radius}" />
+    <joint name="$(arg robot_name)_base_link_right_rear_standoff_joint" type="fixed">
         <origin rpy="0 0 0" xyz="-0.025 -0.125 0.155" />
-        <parent link="base_link" />
-        <child link="right_rear_standoff" />
+        <parent link="$(arg robot_name)_base_link" />
+        <child link="$(arg robot_name)_right_rear_standoff" />
     </joint>
     <!-- cup holder -->
-    <xacro:cup_holder_tray tray_name="cup_holder" tray_length="${cup_holder_length}" tray_radius="${cup_holder_radius}" />
-    <joint name="base_link_cup_holder_joint" type="fixed">
+    <xacro:cup_holder_tray tray_name="$(arg robot_name)_cup_holder" tray_length="${cup_holder_length}" tray_radius="${cup_holder_radius}" />
+    <joint name="$(arg robot_name)_base_link_cup_holder_joint" type="fixed">
         <origin rpy="0 0 0" xyz="0 0 0.42" />
-        <parent link="base_link" />
-        <child link="cup_holder" />
+        <parent link="$(arg robot_name)_base_link" />
+        <child link="$(arg robot_name)_cup_holder" />
     </joint>
     <!-- front caster -->
-    <xacro:caster caster_name="front_caster" caster_length="${caster_length}" caster_radius="${caster_radius}" />
-    <joint name="base_link_front_caster_joint" type="fixed">
+    <xacro:caster caster_name="$(arg robot_name)_front_caster" caster_length="${caster_length}" caster_radius="${caster_radius}" />
+    <joint name="$(arg robot_name)_base_link_front_caster_joint" type="fixed">
         <origin rpy="0 0 0" xyz="0.125 0 0" />
-        <parent link="base_link" />
-        <child link="front_caster" />
+        <parent link="$(arg robot_name)_base_link" />
+        <child link="$(arg robot_name)_front_caster" />
     </joint>
     <!-- rear caster -->
-    <xacro:caster caster_name="rear_caster" caster_length="${caster_length}" caster_radius="${caster_radius}" />
-    <joint name="base_link_rear_caster_joint" type="fixed">
+    <xacro:caster caster_name="$(arg robot_name)_rear_caster" caster_length="${caster_length}" caster_radius="${caster_radius}" />
+    <joint name="$(arg robot_name)_base_link_rear_caster_joint" type="fixed">
         <origin rpy="0 0 0" xyz="-0.125 0 0" />
-        <parent link="base_link" />
-        <child link="rear_caster" />
+        <parent link="$(arg robot_name)_base_link" />
+        <child link="$(arg robot_name)_rear_caster" />
     </joint>
     <!-- laser -->
     <xacro:if value="$(arg include_laser)">
-        <xacro:laser_scanner laser_scanner_name="laser"/>
-        <joint name="base_link_laser_joint" type="fixed">
+        <xacro:laser_scanner laser_scanner_name="$(arg robot_name)_laser"/>
+        <joint name="$(arg robot_name)_base_link_laser_joint" type="fixed">
             <origin rpy="0 0 0" xyz="0 0 0.155" />
-            <parent link="base_link" />
-            <child link="laser" />
+            <parent link="$(arg robot_name)_base_link" />
+            <child link="$(arg robot_name)_laser" />
         </joint>
     </xacro:if>

File: xacro/cup_holder_tray.xacro (robot description, xacro)
@@ -1,4 +1,5 @@
 <?xml version="1.0"?>
 <robot xmlns:xacro="http://www.ros.org/wiki/xacro">
+    <xacro:arg name="tray_color_rviz" default="blue"/>
     <!-- cup holder macro -->
     <xacro:macro name="cup_holder_tray" params="tray_name tray_length tray_radius">
@@ -20,5 +21,5 @@
                     <cylinder length="${tray_length}" radius="${tray_radius}"/>
                 </geometry>
-                <material name="blue"/>
+                <material name="$(arg tray_color_rviz)"/>
             </visual>
         </link>
